File: 4port.brd (EAGLE design)
At the start: 160 x 100 mm, 52 parts, among them IC1 TPS23861PW-HAND, Q1 FDS5680, Q2 FDS5680, Q3 FDS5680, Q4 FDS5680, T1 WE-LAN-10/100/1000-BASE-T,749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, T2 WE-LAN-10/100/1000-BASE-T,749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, X1 22-23-2081

Commit message: foo
Connections:
- net GND: now also LSP1.MP
Changed lines of the file:
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@@
 <contactref element="C3" pad="2"/>
 <contactref element="X1" pad="8"/>
-<wire x1="94.98" y1="69.85" x2="117.8" y2="75.875" width="0" layer="19" extent="1-1"/>
-<wire x1="-34.29" y1="-30.48" x2="94.98" y2="69.85" width="0" layer="19" extent="1-1"/>
+<contactref element="LSP1" pad="MP"/>
+<wire x1="-34.29" y1="-30.48" x2="-52.07" y2="-143.51" width="0" layer="19" extent="1-1"/>
+<wire x1="94.98" y1="69.85" x2="-34.29" y2="-30.48" width="0" layer="19" extent="1-1"/>
+<wire x1="117.8" y1="75.875" x2="94.98" y2="69.85" width="0" layer="19" extent="1-1"/>
 </signal>
 <signal name="N$55">
